File: schematc-io.kicad_sch (KiCad schematic)
At the start: 0 parts

Commit message: First converter version
Parts:
- added C27 (x4): 4n7, Capacitor_SMD:C_1206_3216Metric, symbol Device:C
- added C7 (x2): 100n, Capacitor_SMD:C_1206_3216Metric, symbol Device:C
- added D2, D3, D4: LED, Diode_SMD:D_1206_3216Metric, symbol Device:LED
- added D5: SP0502BAJT, Package_TO_SOT_SMD:SOT-323_SC-70, symbol Power_Protection:SP0502BAJT
- added IC1: AD8544ARUZ-REEL, library:SOP65P640X120-14N, symbol ad8544:AD8544ARUZ-REEL
- added IC2: ACHS-7123-000E, SOIC127P606X204-8N, symbol achs Current Hall Sensor:ACHS-7123-000E
- added R1: 0, LED_SMD:LED_1206_3216Metric, symbol Device:R
- added R17: 60, Resistor_SMD:R_1206_3216Metric, symbol Device:R
- added R18, R2: 10k, LED_SMD:LED_1206_3216Metric, symbol Device:R
- added R18: 150k, LED_SMD:LED_1206_3216Metric, symbol Device:R
- added R18: 60, LED_SMD:LED_1206_3216Metric, symbol Device:R
- added R2, R3, R4: 1k, LED_SMD:LED_1206_3216Metric, symbol Device:R
- added R2: 560k, LED_SMD:LED_1206_3216Metric, symbol Device:R
- added U3: SN65HVD232, Package_SO:SOIC-8_3.9x4.9mm_P1.27mm, symbol Interface_CAN_LIN:SN65HVD232
Connections:
- new net: IC1.12 (+IN_D), R18.1, R18.2
- new net: D4.1 (K), R4.1
- new net: C27.1, R17.1, R18.1
- new net: D3.1 (K), R2.1
- new net: IC2.8 (VDD), R1.2
- new net: D2.1 (K), R3.1
- new net +3.3V: C7.1, C7.1, D4.2 (A), IC1.4 (V+), U3.3 (VCC)
- new net +5V: R1.1
- new net A_Input: IC1.5 (+IN_B), R2.1
- new net Analog_MCU: C27.1, IC1.6 (-IN_B), IC1.7 (OUT_B)
- new net CANH: D5.1 (K), R17.2, U3.7 (CANH)
- new net CANL: D5.2 (K), R18.2, U3.6 (CANL)
- new net CAN_RX: U3.1 (D)
- new net CAN_TX: U3.4 (R)
- new net Current_FC: IC2.7 (VOUT)
- new net FC_Voltage_MCU: C27.2, IC1.13 (-IN_D), IC1.14 (OUT_D)
- new net GND: C27.1, C27.1, C27.2, C27.2, C7.2, C7.2, D5.3 (A), IC1.11 (V-), R18.1, R2.2, R2.2, R2.2, R3.2, R4.2, U3.2 (GND)
- new net LED_CAN_STATUS: D3.2 (A)
- new net LED_MCU_STATUS: D2.2 (A)
- new net SC_V: R18.2
- new net Temp_MCU: C27.2, IC1.1 (OUT_A), IC1.2 (-IN_A)
- new net Temp_sensor: IC1.3 (+IN_A), R2.1
- no-connect marks 0 -> 3
Other:
- note added: "Amplifire"
- note added: "CAN Transceiver"
- note added: "Signal diodes"
- note added: "Termination node (resistors and capacitor) may be omitted during assembly if not required."
- company: (none) -> Hydrogreen Pollub
- title: (none) -> Fuel Cell Control Unit  (FCCU)
