File: schematc-io.kicad_sch (KiCad schematic)
At the start: 23 parts, among them IC1 AD8544ARUZ-REEL, IC2 ACHS-7123-000E, U3 SN65HVD232

Commit message: Repair files
Parts:
- removed C27 (x3): 4n7, Capacitor_SMD:C_1206_3216Metric, symbol Device:C
- removed IC2: ACHS-7123-000E, SOIC127P606X204-8N, symbol achs Current Hall Sensor:ACHS-7123-000E
- removed R1: 0, LED_SMD:LED_1206_3216Metric, symbol Device:R
- removed R18, R2: 10k, LED_SMD:LED_1206_3216Metric, symbol Device:R
- removed R18: 150k, LED_SMD:LED_1206_3216Metric, symbol Device:R
- removed R2: 560k, LED_SMD:LED_1206_3216Metric, symbol Device:R
- added C27 (x3): 4n7, Capacitor_SMD:C_1206_3216Metric, symbol Device:C
- added R18, R2: 10k, LED_SMD:LED_1206_3216Metric, symbol Device:R
- added R18: 150k, LED_SMD:LED_1206_3216Metric, symbol Device:R
- added R2: 560k, LED_SMD:LED_1206_3216Metric, symbol Device:R
Connections:
- net A_Input: now also R2.1
- net Analog_MCU: now also C27.1
- net FC_Voltage_MCU: now also C27.2
- net GND: now also C27.1, C27.1, C27.2, R18.1, R2.2, R2.2
- net Temp_MCU: now also C27.2
- net Temp_sensor: now also R2.1
- net at IC1.12 (+IN_D): now also R18.1, R18.2
- new net FC_V: R18.2
Other:
- note added: "Voltage follower"
- note removed: "Amplifire"

Commit message: P1
Parts:
- removed R18: 10k, LED_SMD:LED_1206_3216Metric, symbol Device:R
- removed R18: 150k, LED_SMD:LED_1206_3216Metric, symbol Device:R
- removed R2: 560k, LED_SMD:LED_1206_3216Metric, symbol Device:R
Connections:
- net FC_V: now also IC1.12 (+IN_D)
- net GND: now also C27.2; no longer C27.1
- net SC_V: now reaches IC1.10 (+IN_C)
- net at IC1.8 (OUT_C): now also C27.1, IC1.9 (-IN_C)
- removed net Temp_MCU: C27.2, IC1.1 (OUT_A), IC1.2 (-IN_A)
- net Temp_sensor: no longer names the net of IC1.3 (+IN_A)
Other:
- moved on the sheet: C7

Commit message: Add test points
Parts:
- added R14, R15: 1k, Resistor_SMD:R_1206_3216Metric, symbol Device:R
- added R2 (x2): 10k, LED_SMD:LED_1206_3216Metric, symbol Device:R
- added R24, R25: 100R, Resistor_SMD:R_1206_3216Metric, symbol Device:R
- added TP1, TP2: GND, symbol Connector:TestPoint
- added TP10: I/O 2, symbol Connector:TestPoint
- added TP11: I/O 3, symbol Connector:TestPoint
- added TP12: I/O 4, symbol Connector:TestPoint
- added TP3, TP4: +12V, symbol Connector:TestPoint
- added TP5, TP6: +5V, symbol Connector:TestPoint
- added TP7, TP8: +3.3V, symbol Connector:TestPoint
- added TP9: I/O 1, symbol Connector:TestPoint
Connections:
- net +12V: now also TP3.1, TP4.1
- net +3.3V: now also TP7.1, TP8.1
- net +5V: now also TP5.1, TP6.1
- net GND: now also R2.2, R2.2, TP1.1, TP2.1
- new net: R14.1, TP9.1
- new net: R24.1, TP11.1
- new net: R25.1, TP12.1
- new net: R15.1, TP10.1
- new net I/O_1_MCU: R14.2
- new net I/O_2_MCU: R15.2
- new net I/O_3_MCU: R2.1, R24.2
- new net I/O_4_MCU: R2.1, R25.2
Other:
- note added: "Test points"

Commit message: Edit mosfets outputs
Parts:
- removed C27 (x3): 4n7, Capacitor_SMD:C_1206_3216Metric, symbol Device:C
- removed R2: 10k, LED_SMD:LED_1206_3216Metric, symbol Device:R
- added C27 (x2): 4n7, Capacitor_SMD:C_1206_3216Metric, symbol Device:C
Connections:
- net A_Input is gone; now on net SC_V: IC1.5 (+IN_B)
- net FC_V: now also IC1.10 (+IN_C); no longer IC1.12 (+IN_D)
- net FC_Voltage_MCU: now also IC1.8 (OUT_C), IC1.9 (-IN_C), C27.1; no longer IC1.13 (-IN_D), IC1.14 (OUT_D)
- net GND: now also C27.2, C27.2
- net SC_V: no longer IC1.10 (+IN_C)
- net Analog_MCU renamed SC_Voltage_MCU
- net SC_Voltage_MCU: now also C27.1
- no-connect marks 3 -> 6

Commit message: First pcb
Parts:
- TP1, TP10, TP11, TP12, TP2, TP3, TP4, TP5, TP6, TP7, TP8, TP9: footprint (none) -> Connector_PinSocket_2.54mm:PinSocket_1x01_P2.54mm_Vertical
- renumbered IC1 to IC2, R14 to R20, R15 to R21, R24 to R22, R25 to R23

Commit message: Buck - boost converter
Parts:
- added R43: 100R, Resistor_SMD:R_1206_3216Metric, symbol Device:R
- added R44: 10k, LED_SMD:LED_1206_3216Metric, symbol Device:R
- added TP20: I/O 4, Connector_PinSocket_2.54mm:PinSocket_1x01_P2.54mm_Vertical, symbol Connector:TestPoint
- renumbered C27 to C29, C7 to C31, R2 to R24, R2 to R25
Connections:
- net GND: now also R44.2
- net I/O_4_MCU: now also R43.2, R44.1
- new net: R43.1, TP20.1
Other:
- note added: "Sterowanie potencjometrami cyfrowymi dodatkowej przetwornicy"

Commit message: Add pot
Parts:
- removed TP20: I/O 4, Connector_PinSocket_2.54mm:PinSocket_1x01_P2.54mm_Vertical, symbol Connector:TestPoint
- added C50: 100n, Capacitor_SMD:C_1206_3216Metric, symbol Device:C
- added IC8: MCP4018T-503E_LT, SOT65P210X110-6N, symbol digital pot 100k:MCP4018T-503E_LT
- added R52, R53: 10k, LED_SMD:LED_1206_3216Metric, symbol Device:R
- added R54, R55: 4,7k, LED_SMD:LED_1206_3216Metric, symbol Device:R
- added TP23: D_Pot_W, Connector_PinSocket_2.54mm:PinSocket_1x01_P2.54mm_Vertical, symbol Connector:TestPoint
- added TP24: D_Pot_A, Connector_PinSocket_2.54mm:PinSocket_1x01_P2.54mm_Vertical, symbol Connector:TestPoint
- R43: value 100R -> 10k; footprint Resistor_SMD:R_1206_3216Metric -> LED_SMD:LED_1206_3216Metric
Connections:
- net +3.3V: now also C50.1, IC8.1 (VDD), R53.1, R54.1, R55.1
- net GND: now also R43.2, C50.2, IC8.2 (VSS); no longer R44.2
- net I/O_4_MCU: no longer R43.2, R44.1
- net at R43.1: now also R44.2, TP23.1
- new net: IC8.5 (W), R44.1
- new net: R52.1, R53.2, TP24.1
- new net: IC8.6 (A), R52.2
- new net SCL_D_Pot_i2c_MCU: IC8.3 (SCL), R55.2
- new net SDA_D_Pot_i2c_MCU: IC8.4 (SDA), R54.2
Other:
- note added: "Rezystory do wyboru w zależności od zastosowania A - wejście na potencjometr W - wyjście środka potencjometru VSS - doł potencjometru na gnd"

Commit message: PCB design 80%
Parts:
- IC8: footprint SOT65P210X110-6N -> Lib:SOT65P210X110-6N
- R18, R2, R24, R25, R3, R4, R43, R44, R52, R53, R54, R55: footprint LED_SMD:LED_1206_3216Metric -> Resistor_SMD:R_1206_3216Metric
Changed lines of the file:
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@@
 			)
 		)
-		(property "Footprint" "LED_SMD:LED_1206_3216Metric"
+		(property "Footprint" "Resistor_SMD:R_1206_3216Metric"
 			(at 261.62 130.937 90)
 			(effects
@@
 			)
 		)
-		(property "Footprint" "LED_SMD:LED_1206_3216Metric"
+		(property "Footprint" "Resistor_SMD:R_1206_3216Metric"
 			(at 128.016 185.547 90)
 			(effects
@@
 			)
 		)
-		(property "Footprint" "LED_SMD:LED_1206_3216Metric"
+		(property "Footprint" "Resistor_SMD:R_1206_3216Metric"
 			(at 261.62 123.317 90)
 			(effects
@@
 			)
 		)
-		(property "Footprint" "LED_SMD:LED_1206_3216Metric"
+		(property "Footprint" "Resistor_SMD:R_1206_3216Metric"
 			(at 256.413 112.649 90)
 			(effects
@@
 			)
 		)
-		(property "Footprint" "LED_SMD:LED_1206_3216Metric"
+		(property "Footprint" "Resistor_SMD:R_1206_3216Metric"
 			(at 255.143 78.105 90)
 			(effects
@@
 			)
 		)
-		(property "Footprint" "LED_SMD:LED_1206_3216Metric"
+		(property "Footprint" "Resistor_SMD:R_1206_3216Metric"
 			(at 153.416 185.547 90)
 			(effects
@@
 			)
 		)
-		(property "Footprint" "SOT65P210X110-6N"
+		(property "Footprint" "Lib:SOT65P210X110-6N"
 			(at 231.775 211.506 0)
 			(effects
@@
 			)
 		)
-		(property "Footprint" "LED_SMD:LED_1206_3216Metric"
+		(property "Footprint" "Resistor_SMD:R_1206_3216Metric"
 			(at 199.263 139.827 90)
 			(effects
@@
 			)
 		)
-		(property "Footprint" "LED_SMD:LED_1206_3216Metric"
+		(property "Footprint" "Resistor_SMD:R_1206_3216Metric"
 			(at 207.772 144.018 90)
 			(effects
@@
 			)
 		)
-		(property "Footprint" "LED_SMD:LED_1206_3216Metric"
+		(property "Footprint" "Resistor_SMD:R_1206_3216Metric"
 			(at 140.716 185.547 90)
 			(effects
@@
 			)
 		)
-		(property "Footprint" "LED_SMD:LED_1206_3216Metric"
+		(property "Footprint" "Resistor_SMD:R_1206_3216Metric"
 			(at 256.413 105.029 90)
 			(effects
@@
 			)
 		)
-		(property "Footprint" "LED_SMD:LED_1206_3216Metric"
+		(property "Footprint" "Resistor_SMD:R_1206_3216Metric"
 			(at 121.285 62.992 90)
 			(effects
@@
 			)
 		)
-		(property "Footprint" "LED_SMD:LED_1206_3216Metric"
+		(property "Footprint" "Resistor_SMD:R_1206_3216Metric"
 			(at 255.143 60.325 90)
 			(effects
