File: schematic-main.kicad_sch (KiCad schematic)
At the start: 44 parts, among them J1 Conn_01x02_Socket, J4 Conn_01x02_Pin, P1 USB_C_Plug_USB2.0, SW1 SW_Push, SW2 SW_Push, U2 MQ-8, U3 SN65HVD232, U5 USBLC6-2P6, U6 ESP32-S3FN8, Y1 Crystal_GND24

Commit message: First converter version
Parts:
- removed C1, C30, C31, C34, C6, C7, C8: 100n, symbol Device:C
- removed C2, C28, C33, C35: 1u, symbol Device:C
- removed C27: 4n7, symbol Device:C
- removed C29: 10n, symbol Device:C
- removed C32: 10u, symbol Device:C
- removed C4, C5: 12p, symbol Device:C
- removed D2, D3, D4: LED, symbol Device:LED
- removed D5: SP0502BAJT, Package_TO_SOT_SMD:SOT-323_SC-70, symbol Power_Protection:SP0502BAJT
- removed D6: D, symbol Device:D
- removed J1: Conn_01x02_Socket, symbol Connector:Conn_01x02_Socket
- removed J4: Conn_01x02_Pin, symbol Connector:Conn_01x02_Pin
- removed L3: 2n, symbol Device:L
- removed R17, R18: 60, symbol Device:R
- removed R19, R22: 5k1, symbol Device:R
- removed R20, R21: 0, symbol Device:R
- removed R23, R5: 10k, symbol Device:R
- removed SW1, SW2: SW_Push, symbol Switch:SW_Push
- removed U2: MQ-8, Sensor:MQ-6, symbol Sensor_Gas:MQ-6
- removed U3: SN65HVD232, Package_SO:SOIC-8_3.9x4.9mm_P1.27mm, symbol Interface_CAN_LIN:SN65HVD232
- removed U5: USBLC6-2P6, Package_TO_SOT_SMD:SOT-666, symbol Power_Protection:USBLC6-2P6
- removed U6: ESP32-S3FN8, Package_DFN_QFN:QFN-56-1EP_7x7mm_P0.4mm_EP5.6x5.6mm, symbol PCM_Espressif:ESP32-S3
- removed Y1: Crystal_GND24, symbol Device:Crystal_GND24
- added J1: Fell_Cell_IN, Connector_Molex:Molex_Mini-Fit_Jr_5569-02A2_2x01_P4.20mm_Horizontal, symbol Connector:Conn_01x02_Pin
- added J2: CAN, Connector_Molex:Molex_Mini-Fit_Jr_5569-02A2_2x01_P4.20mm_Horizontal, symbol Connector_Generic:Conn_01x02
- added J3: P_Valve, Connector_Molex:Molex_Mini-Fit_Jr_5569-02A2_2x01_P4.20mm_Horizontal, symbol Connector_Generic:Conn_01x02
- added J4: FC Cooling, Connector_Molex:Molex_Mini-Fit_Jr_5569-10A1_2x05_P4.20mm_Horizontal, symbol Connector_Generic:Conn_02x05_Top_Bottom
- added J5: Valve, Connector_Molex:Molex_Mini-Fit_Jr_5569-02A2_2x01_P4.20mm_Horizontal, symbol Connector_Generic:Conn_01x02
- added J7: Axilary_Out, Connector_Molex:Molex_Mini-Fit_Jr_5569-02A2_2x01_P4.20mm_Horizontal, symbol Connector_Generic:Conn_01x02
- added J9: Analog_In, Connector_Molex:Molex_Mini-Fit_Jr_5569-02A2_2x01_P4.20mm_Horizontal, symbol Connector_Generic:Conn_01x02
- P1: footprint (none) -> library:2169900002
- R1: value 10k -> 0; footprint (none) -> Resistor_SMD:R_1206_3216Metric
- R2: value 1k -> 0; footprint (none) -> Resistor_SMD:R_1206_3216Metric
- R3, R4: value 1k -> 5k1; footprint (none) -> Resistor_SMD:R_1206_3216Metric
Connections:
- net SENSOR_ADC is gone; now on an unnamed net: R1.1
- net +3.3V: now also J4.10 (Pin_10), J9.1 (Pin_1)
- net GND: now also J1.2 (Pin_2), J7.2 (Pin_2); no longer R1.2, R2.2
- net Power /Vin: now also J1.1 (Pin_1)
- net at P1.B5 (VCONN): now also R3.1
- net VBUS: now reaches P1.A4 (VBUS), P1.A9 (VBUS), P1.B4 (VBUS), P1.B9 (VBUS)
- net at R2.1: now also P1.A6 (D+)
- net at P1.A5 (CC): now also R4.1
- new net +12V: J3.1 (Pin_1), J4.1 (Pin_1), J4.6 (Pin_6), J5.1 (Pin_1)
- new net IO/A_Input: J9.2 (Pin_2)
- new net IO/CANH: J2.1 (Pin_1)
- new net IO/CANL: J2.2 (Pin_2)
- new net IO/FAN_1_TACHO: J4.3 (Pin_3)
- new net IO/FAN_2_TACHO: J4.8 (Pin_8)
- new net IO/FAN_GND: J4.4 (Pin_4), J4.9 (Pin_9)
- new net IO/FAN_PWM: J4.2 (Pin_2), J4.7 (Pin_7)
- new net IO/Main_Valve: J5.2 (Pin_2)
- new net IO/PURGE_VALVE: J3.2 (Pin_2)
- new net IO/Temp_sensor: J4.5 (Pin_5)
- new net IO/out_12V: J7.1 (Pin_1)
- new net MCU/USB_D+: R2.2
- new net MCU/USB_D-: R1.2
- no-connect marks 3 -> 0
Other:
- added sheet MCU (schematic-mcu.kicad_sch)
- added sheet Step Down Converter (schematc-converter.kicad_sch)
- sheet IO ports: added 12V, 3.3V, A_Input, Analog_MCU, CANH, CANL, CAN_RX, CAN_TX, FAN_1_TACHO, FAN_1_TACHO_MCU, FAN_2_TACHO, FAN_2_TACHO_MCU, FAN_GND, FAN_ON_MCU, FAN_PWM, FAN_PWM_MCU, FC_Voltage_MCU, GND, LED_CAN_STATUS, LED_MCU_STATUS, Main_Valve, Main_Valve_MCU, PURGE_VALVE, PURGE_VALVE_MCU, SC_V, Temp_MCU, Temp_sensor, out_12V; removed none
- sheet Power  ports: added GND, SC_V, VBUS; removed +5V
- note added: "30-62V"
- note removed: "Boot button"
- note removed: "CAN Transceiver"
- note removed: "C_{x} = (C_{load} - C_{stray}) * 2 = = (8 pF - 2 pF) * 2 = 12 pF"
- note removed: "Crystal oscillator"
- note removed: "Hydrogen sensor"
- note removed: "I_{max}: 250 mA P_{max}: 800 mW"
- note removed: "Microcontroller"
- note removed: "Power section"
- note removed: "Reset button"
- note removed: "Signal diodes"
- note removed: "TODO Protect USB reverse-polarity Ensure MCU receive 3.3 V from USB-C"
- note removed: "TODO: Add diode's pinout Update component numeration"
- note removed: "Termination node (resistors and capacitor) may be omitted during assembly if not required."
- note removed: "USB-C (programming and debugging)"
- title: Hydrogen sensor -> Fuel Cell Control Unit  (FCCU)
