File: schematc-converter.kicad_sch (KiCad schematic)
At the start: 69 parts, among them IC2 ACHS-7121-000E, IC2 ACHS-7123-000E, IC6 LM5106MMX_NOPB, IC7 LM5106MMX_NOPB, Q1 CSD19531Q5AT, Q2 CSD19531Q5AT, Q3 CSD19531Q5AT, Q4 CSD19531Q5AT

Commit message: PCB design 80%
Parts:
- D10, D11, D12, D7, D8, D9: footprint SODFL3718X170N -> Lib:SODFL3718X170N
- IC2: footprint SOIC127P606X204-8N -> Lib:SOIC127P606X204-8N
- IC6, IC7: footprint SOP50P490X110-10N -> Lib:SOP50P490X110-10N
- Q1, Q2, Q3, Q4: footprint CSD19531Q5AT -> Lib:CSD19531Q5AT
- R18, R2, R46, R48, R49: footprint LED_SMD:LED_1206_3216Metric -> Resistor_SMD:R_1206_3216Metric
- R18, R45, R47: footprint LED_SMD:LED_1206_3216Metric -> Resistor_SMD:R_2512_6332Metric
- R50, R51: footprint LED_SMD:LED_1206_3216Metric -> Resistor_SMD:R_2512_6332Metric_Pad1.40x3.35mm_HandSolder
Changed lines of the file:
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@@
 			)
 		)
-		(property "Footprint" "LED_SMD:LED_1206_3216Metric"
+		(property "Footprint" "Resistor_SMD:R_1206_3216Metric"
 			(at 80.137 112.395 90)
 			(effects
@@
 			)
 		)
-		(property "Footprint" "LED_SMD:LED_1206_3216Metric"
+		(property "Footprint" "Resistor_SMD:R_1206_3216Metric"
 			(at 78.867 147.32 90)
 			(effects
@@
 			)
 		)
-		(property "Footprint" "LED_SMD:LED_1206_3216Metric"
+		(property "Footprint" "Resistor_SMD:R_1206_3216Metric"
 			(at 80.137 120.015 90)
 			(effects
@@
 			)
 		)
-		(property "Footprint" "LED_SMD:LED_1206_3216Metric"
+		(property "Footprint" "Resistor_SMD:R_1206_3216Metric"
 			(at 227.838 40.64 90)
 			(effects
@@
 			)
 		)
-		(property "Footprint" "LED_SMD:LED_1206_3216Metric"
+		(property "Footprint" "Resistor_SMD:R_1206_3216Metric"
 			(at 247.015 155.067 90)
 			(effects
@@
 			)
 		)
-		(property "Footprint" "SODFL3718X170N"
+		(property "Footprint" "Lib:SODFL3718X170N"
 			(at 229.87 135.255 0)
 			(effects
@@
 			)
 		)
-		(property "Footprint" "CSD19531Q5AT"
+		(property "Footprint" "Lib:CSD19531Q5AT"
 			(at 127.635 -23.8 0)
 			(effects
@@
 			)
 		)
-		(property "Footprint" "SOP50P490X110-10N"
+		(property "Footprint" "Lib:SOP50P490X110-10N"
 			(at 209.55 242.24 0)
 			(effects
@@
 			)
 		)
-		(property "Footprint" "LED_SMD:LED_1206_3216Metric"
+		(property "Footprint" "Resistor_SMD:R_2512_6332Metric_Pad1.40x3.35mm_HandSolder"
 			(at 110.49 42.672 90)
 			(effects
@@
 			)
 		)
-		(property "Footprint" "LED_SMD:LED_1206_3216Metric"
+		(property "Footprint" "Resistor_SMD:R_2512_6332Metric"
 			(at 157.48 154.178 90)
 			(effects
@@
 			)
 		)
-		(property "Footprint" "SODFL3718X170N"
+		(property "Footprint" "Lib:SODFL3718X170N"
 			(at 157.48 160.02 0)
 			(effects
@@
 			)
 		)
-		(property "Footprint" "LED_SMD:LED_1206_3216Metric"
+		(property "Footprint" "Resistor_SMD:R_1206_3216Metric"
 			(at 84.582 48.895 90)
 			(effects
@@
 			)
 		)
-		(property "Footprint" "LED_SMD:LED_1206_3216Metric"
+		(property "Footprint" "Resistor_SMD:R_1206_3216Metric"
 			(at 77.597 182.245 90)
 			(effects
@@
 			)
 		)
-		(property "Footprint" "SODFL3718X170N"
+		(property "Footprint" "Lib:SODFL3718X170N"
 			(at 227.33 87.63 0)
 			(effects
@@
 			)
 		)
-		(property "Footprint" "LED_SMD:LED_1206_3216Metric"
+		(property "Footprint" "Resistor_SMD:R_1206_3216Metric"
 			(at 216.027 114.935 90)
 			(effects
@@
 			)
 		)
-		(property "Footprint" "LED_SMD:LED_1206_3216Metric"
+		(property "Footprint" "Resistor_SMD:R_2512_6332Metric"
 			(at 158.75 107.188 90)
 			(effects
@@
 			)
 		)
-		(property "Footprint" "SOIC127P606X204-8N"
+		(property "Footprint" "Lib:SOIC127P606X204-8N"
 			(at 53.34 268.91 0)
 			(effects
@@
 			)
 		)
-		(property "Footprint" "LED_SMD:LED_1206_3216Metric"
+		(property "Footprint" "Resistor_SMD:R_2512_6332Metric"
 			(at 229.87 140.208 90)
 			(effects
@@
 			)
 		)
-		(property "Footprint" "LED_SMD:LED_1206_3216Metric"
+		(property "Footprint" "Resistor_SMD:R_1206_3216Metric"
 			(at 227.838 52.07 90)
 			(effects
@@
 			)
 		)
-		(property "Footprint" "LED_SMD:LED_1206_3216Metric"
+		(property "Footprint" "Resistor_SMD:R_1206_3216Metric"
 			(at 214.757 161.925 90)
 			(effects
@@
 			)
 		)
-		(property "Footprint" "CSD19531Q5AT"
+		(property "Footprint" "Lib:CSD19531Q5AT"
 			(at 182.88 -22.53 0)
 			(effects
@@
 			)
 		)
-		(property "Footprint" "LED_SMD:LED_1206_3216Metric"
+		(property "Footprint" "Resistor_SMD:R_2512_6332Metric"
 			(at 159.512 67.31 90)
 			(effects
@@
 			)
 		)
-		(property "Footprint" "LED_SMD:LED_1206_3216Metric"
+		(property "Footprint" "Resistor_SMD:R_1206_3216Metric"
 			(at 249.555 154.178 90)
 			(effects
@@
 			)
 		)
-		(property "Footprint" "LED_SMD:LED_1206_3216Metric"
+		(property "Footprint" "Resistor_SMD:R_1206_3216Metric"
 			(at 78.867 154.94 90)
 			(effects
@@
 			)
 		)
-		(property "Footprint" "LED_SMD:LED_1206_3216Metric"
+		(property "Footprint" "Resistor_SMD:R_1206_3216Metric"
 			(at 77.597 189.865 90)
 			(effects
@@
 			)
 		)
-		(property "Footprint" "LED_SMD:LED_1206_3216Metric"
+		(property "Footprint" "Resistor_SMD:R_1206_3216Metric"
 			(at 84.582 37.465 90)
 			(effects
@@
 			)
 		)
-		(property "Footprint" "LED_SMD:LED_1206_3216Metric"
+		(property "Footprint" "Resistor_SMD:R_2512_6332Metric_Pad1.40x3.35mm_HandSolder"
 			(at 200.66 41.402 90)
 			(effects
@@
 			)
 		)
-		(property "Footprint" "LED_SMD:LED_1206_3216Metric"
+		(property "Footprint" "Resistor_SMD:R_1206_3216Metric"
 			(at 248.285 108.077 90)
 			(effects
@@
 			)
 		)
-		(property "Footprint" "CSD19531Q5AT"
+		(property "Footprint" "Lib:CSD19531Q5AT"
 			(at 200.66 -56.82 0)
 			(effects
@@
 			)
 		)
-		(property "Footprint" "LED_SMD:LED_1206_3216Metric"
+		(property "Footprint" "Resistor_SMD:R_2512_6332Metric"
 			(at 159.512 41.91 90)
 			(effects
@@
 			)
 		)
-		(property "Footprint" "SODFL3718X170N"
+		(property "Footprint" "Lib:SODFL3718X170N"
 			(at 158.75 113.03 0)
 			(effects
@@
 			)
 		)
-		(property "Footprint" "CSD19531Q5AT"
+		(property "Footprint" "Lib:CSD19531Q5AT"
 			(at 109.855 -54.915 0)
 			(effects
@@
 			)
 		)
-		(property "Footprint" "LED_SMD:LED_1206_3216Metric"
+		(property "Footprint" "Resistor_SMD:R_1206_3216Metric"
 			(at 250.825 107.188 90)
 			(effects
@@
 			)
 		)
-		(property "Footprint" "SODFL3718X170N"
+		(property "Footprint" "Lib:SODFL3718X170N"
 			(at 183.515 97.155 0)
 			(effects
@@
 			)
 		)
-		(property "Footprint" "LED_SMD:LED_1206_3216Metric"
+		(property "Footprint" "Resistor_SMD:R_2512_6332Metric"
 			(at 227.33 92.583 90)
 			(effects
@@
 			)
 		)
-		(property "Footprint" "SODFL3718X170N"
+		(property "Footprint" "Lib:SODFL3718X170N"
 			(at 182.245 144.145 0)
 			(effects
@@
 			)
 		)
-		(property "Footprint" "SOIC127P606X204-8N"
+		(property "Footprint" "Lib:SOIC127P606X204-8N"
 			(at 55.88 199.06 0)
 			(effects
@@
 			)
 		)
-		(property "Footprint" "SOP50P490X110-10N"
+		(property "Footprint" "Lib:SOP50P490X110-10N"
 			(at 210.82 195.25 0)
 			(effects
@@
 			)
 		)
-		(property "Footprint" "SOIC127P606X204-8N"
+		(property "Footprint" "Lib:SOIC127P606X204-8N"
 			(at 54.61 233.985 0)
 			(effects
