File: schematc-converter.kicad_sch (KiCad schematic)
At the start: 69 parts, among them IC2 ACHS-7121-000E, IC2 ACHS-7123-000E, IC6 LM5106MMX_NOPB, IC7 LM5106MMX_NOPB, Q1 CSD19531Q5AT, Q2 CSD19531Q5AT, Q3 CSD19531Q5AT, Q4 CSD19531Q5AT

Commit message: PCB design complate
Parts:
- TP17: value EN test -> EN A test
- TP18: value PWM test -> PWM A test
- TP21: value EN test -> EN B test
- TP22: value PWM test -> PWM B test
Connections:
- net Converter_ON_B_MCU: no longer R2.1
- net Converter_PWM_B_MCU: no longer R2.2
- new net Converter_ON_A_MCU: R2.1
- new net Converter_PWM_A_MCU: R2.2
Changed lines of the file:
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@@
 		)
 	)
-	(hierarchical_label "Converter_ON_B_MCU"
+	(hierarchical_label "Converter_ON_A_MCU"
 		(shape input)
 		(at 255.27 109.855 0)
@@
 		)
 	)
-	(hierarchical_label "Converter_PWM_B_MCU"
+	(hierarchical_label "Converter_PWM_A_MCU"
 		(shape input)
 		(at 257.175 105.41 0)
@@
 		(fields_autoplaced yes)
 		(property "Reference" "TP18"
-			(at 234.315 100.838 0)
+			(at 234.95 100.8379 0)
 			(effects
 				(font
@@
 			)
 		)
-		(property "Value" "PWM test"
-			(at 234.315 103.378 0)
+		(property "Value" "PWM A test"
+			(at 234.95 103.3779 0)
 			(effects
 				(font
@@
 		(fields_autoplaced yes)
 		(property "Reference" "TP22"
-			(at 233.045 147.828 0)
+			(at 233.68 147.8279 0)
 			(effects
 				(font
@@
 			)
 		)
-		(property "Value" "PWM test"
-			(at 233.045 150.368 0)
+		(property "Value" "PWM B test"
+			(at 233.68 150.3679 0)
 			(effects
 				(font
@@
 		(fields_autoplaced yes)
 		(property "Reference" "TP17"
-			(at 234.315 111.887 0)
+			(at 233.68 111.8869 0)
 			(effects
 				(font
@@
 			)
 		)
-		(property "Value" "EN test"
-			(at 234.315 114.427 0)
+		(property "Value" "EN A test"
+			(at 233.68 114.4269 0)
 			(effects
 				(font
@@
 		(fields_autoplaced yes)
 		(property "Reference" "TP21"
-			(at 233.045 158.877 0)
+			(at 232.41 158.8769 0)
 			(effects
 				(font
@@
 			)
 		)
-		(property "Value" "EN test"
-			(at 233.045 161.417 0)
+		(property "Value" "EN B test"
+			(at 232.41 161.4169 0)
 			(effects
 				(font
