File: schematic-mcu.kicad_sch (KiCad schematic)
At the start: 28 parts, among them U5 USBLC6-2P6, U6 ESP32-S3FN8, Y1 Crystal_GND24

Commit message: Repair files
Parts:
- removed R23 (x3): 10k, LED_SMD:LED_1206_3216Metric, symbol Device:R
Changed lines of the file:
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@@
   (junction (at 175.26 53.34) (diameter 0) (color 0 0 0 0)
   )
-  (junction (at 135.382 145.034) (diameter 0) (color 0 0 0 0)
-  )
   (junction (at 163.83 53.34) (diameter 0) (color 0 0 0 0)
   )
@@
   (junction (at 185.928 152.019) (diameter 0) (color 0 0 0 0)
   )
-  (junction (at 141.351 125.984) (diameter 0) (color 0 0 0 0)
-  )
   (junction (at 31.75 45.72) (diameter 0) (color 0 0 0 0)
   )
@@
   )
   (junction (at 246.38 53.34) (diameter 0) (color 0 0 0 0)
-  )
-  (junction (at 172.847 110.236) (diameter 0) (color 0 0 0 0)
   )
   (no_connect (at 261.62 77.47))
@@
     (stroke (width 0) (type default))
   )
-  (wire (pts (xy 138.811 125.984) (xy 141.351 125.984))
-    (stroke (width 0) (type default))
-  )
   (wire (pts (xy 95.25 49.53) (xy 95.25 50.8))
     (stroke (width 0) (type default))
@@
     (stroke (width 0) (type default))
   )
-  (wire (pts (xy 172.847 110.236) (xy 176.911 110.236))
-    (stroke (width 0) (type default))
-  )
   (wire (pts (xy 176.911 110.236) (xy 176.911 118.11))
     (stroke (width 0) (type default))
@@
     (stroke (width 0) (type default))
   )
-  (wire (pts (xy 166.497 110.236) (xy 172.847 110.236))
+  (wire (pts (xy 166.497 110.236) (xy 176.911 110.236))
     (stroke (width 0) (type default))
   )
@@
     (stroke (width 0) (type default))
   )
-  (wire (pts (xy 135.382 136.144) (xy 135.382 137.414))
-    (stroke (width 0) (type default))
-  )
   (wire (pts (xy 62.611 114.427) (xy 62.611 109.347))
     (stroke (width 0) (type default))
@@
     (stroke (width 0) (type default))
   )
-  (wire (pts (xy 141.605 125.984) (xy 141.605 125.73))
-    (stroke (width 0) (type default))
-  )
   (wire (pts (xy 212.09 38.1) (xy 212.09 39.37))
     (stroke (width 0) (type default))
@@
     (stroke (width 0) (type default))
   )
-  (wire (pts (xy 141.351 117.094) (xy 141.351 118.364))
-    (stroke (width 0) (type default))
-  )
   (wire (pts (xy 46.101 100.457) (xy 46.101 111.887))
     (stroke (width 0) (type default))
@@
     (stroke (width 0) (type default))
   )
-  (wire (pts (xy 135.382 145.034) (xy 153.289 145.034))
+  (wire (pts (xy 132.842 145.034) (xy 153.289 145.034))
     (stroke (width 0) (type default))
   )
@@
     (stroke (width 0) (type default))
   )
-  (wire (pts (xy 141.351 125.984) (xy 141.605 125.984))
+  (wire (pts (xy 139.7 125.73) (xy 195.58 125.73))
     (stroke (width 0) (type default))
   )
@@
     (stroke (width 0) (type default))
   )
-  (wire (pts (xy 132.842 145.034) (xy 135.382 145.034))
-    (stroke (width 0) (type default))
-  )
   (wire (pts (xy 95.25 40.64) (xy 95.25 41.91))
     (stroke (width 0) (type default))
@@
     (stroke (width 0) (type default))
   )
-  (wire (pts (xy 169.037 102.616) (xy 172.847 102.616))
-    (stroke (width 0) (type default))
-  )
   (wire (pts (xy 43.18 40.64) (xy 43.18 41.91))
     (stroke (width 0) (type default))
@@
   )
   (wire (pts (xy 59.309 154.559) (xy 59.309 153.289))
-    (stroke (width 0) (type default))
-  )
-  (wire (pts (xy 141.605 125.73) (xy 195.58 125.73))
     (stroke (width 0) (type default))
   )
@@
     (effects (font (size 1.27 1.27)) (justify right))
   )
-  (hierarchical_label "FAN_1_TACHO_MCU" (shape input) (at 138.811 125.984 180) (fields_autoplaced)
+  (hierarchical_label "FAN_1_TACHO_MCU" (shape input) (at 139.7 125.73 180) (fields_autoplaced)
     (effects (font (size 1.27 1.27)) (justify right))
   )
@@
     )
   )
-  (symbol (lib_id "power:+3.3V") (at 135.382 136.144 0) (unit 1)
-    (in_bom yes) (on_board yes) (dnp no) (fields_autoplaced)
-    (property "Reference" "#PWR02" (at 135.382 139.954 0)
-      (effects (font (size 1.27 1.27)) hide)
-    )
-    (property "Value" "+3.3V" (at 135.382 131.699 0)
-      (effects (font (size 1.27 1.27)))
-    )
-    (property "Footprint" "" (at 135.382 136.144 0)
-      (effects (font (size 1.27 1.27)) hide)
-    )
-    (property "Datasheet" "" (at 135.382 136.144 0)
-      (effects (font (size 1.27 1.27)) hide)
-    )
-    (pin "1")
-    (instances
-      (project "schematic-main"
-        (path "/c9ad7189-d3b2-414a-9743-efd8e57cd755"
-          (reference "#PWR02") (unit 1)
-        )
-        (path "/c9ad7189-d3b2-414a-9743-efd8e57cd755/f92f58ec-64e0-437c-bc00-8ae46a3b3054"
-          (reference "#PWR063") (unit 1)
-        )
-      )
-    )
-  )
   (symbol (lib_id "Device:L") (at 194.31 53.34 90) (unit 1)
     (in_bom yes) (on_board yes) (dnp no) (fields_autoplaced)
@@
     )
   )
-  (symbol (lib_id "power:+3.3V") (at 141.351 117.094 0) (unit 1)
-    (in_bom yes) (on_board yes) (dnp no) (fields_autoplaced)
-    (property "Reference" "#PWR02" (at 141.351 120.904 0)
-      (effects (font (size 1.27 1.27)) hide)
-    )
-    (property "Value" "+3.3V" (at 141.351 112.649 0)
-      (effects (font (size 1.27 1.27)))
-    )
-    (property "Footprint" "" (at 141.351 117.094 0)
-      (effects (font (size 1.27 1.27)) hide)
-    )
-    (property "Datasheet" "" (at 141.351 117.094 0)
-      (effects (font (size 1.27 1.27)) hide)
-    )
-    (pin "1")
-    (instances
-      (project "schematic-main"
-        (path "/c9ad7189-d3b2-414a-9743-efd8e57cd755"
-          (reference "#PWR02") (unit 1)
-        )
-        (path "/c9ad7189-d3b2-414a-9743-efd8e57cd755/f92f58ec-64e0-437c-bc00-8ae46a3b3054"
-          (reference "#PWR062") (unit 1)
-        )
-      )
-    )
-  )
   (symbol (lib_id "Device:C") (at 45.339 165.989 0) (unit 1)
     (in_bom yes) (on_board yes) (dnp no) (fields_autoplaced)
@@
     )
   )
-  (symbol (lib_id "power:GND") (at 169.037 102.616 0) (unit 1)
-    (in_bom yes) (on_board yes) (dnp no) (fields_autoplaced)
-    (property "Reference" "#PWR053" (at 169.037 108.966 0)
-      (effects (font (size 1.27 1.27)) hide)
-    )
-    (property "Value" "GND" (at 169.037 107.696 0)
-      (effects (font (size 1.27 1.27)) hide)
-    )
-    (property "Footprint" "" (at 169.037 102.616 0)
-      (effects (font (size 1.27 1.27)) hide)
-    )
-    (property "Datasheet" "" (at 169.037 102.616 0)
-      (effects (font (size 1.27 1.27)) hide)
-    )
-    (pin "1")
-    (instances
-      (project "schematic-main"
-        (path "/c9ad7189-d3b2-414a-9743-efd8e57cd755"
-          (reference "#PWR053") (unit 1)
-        )
-        (path "/c9ad7189-d3b2-414a-9743-efd8e57cd755/e4695f4d-6fa6-4597-a598-6a2f28a255eb"
-          (reference "#PWR047") (unit 1)
-        )
-        (path "/c9ad7189-d3b2-414a-9743-efd8e57cd755/f92f58ec-64e0-437c-bc00-8ae46a3b3054"
-          (reference "#PWR064") (unit 1)
-        )
-      )
-    )
-  )
   (symbol (lib_id "power:GND") (at 256.54 66.04 0) (unit 1)
     (in_bom yes) (on_board yes) (dnp no) (fields_autoplaced)
@@
         (path "/c9ad7189-d3b2-414a-9743-efd8e57cd755/f92f58ec-64e0-437c-bc00-8ae46a3b3054"
           (reference "#PWR027") (unit 1)
-        )
-      )
-    )
-  )
-  (symbol (lib_id "Device:R") (at 172.847 106.426 180) (unit 1)
-    (in_bom yes) (on_board yes) (dnp no) (fields_autoplaced)
-    (property "Reference" "R23" (at 174.752 105.1559 0)
-      (effects (font (size 1.27 1.27)) (justify right))
-    )
-    (property "Value" "10k" (at 174.752 107.6959 0)
-      (effects (font (size 1.27 1.27)) (justify right))
-    )
-    (property "Footprint" "LED_SMD:LED_1206_3216Metric" (at 174.625 106.426 90)
-      (effects (font (size 1.27 1.27)) hide)
-    )
-    (property "Datasheet" "~" (at 172.847 106.426 0)
-      (effects (font (size 1.27 1.27)) hide)
-    )
-    (pin "1")
-    (pin "2")
-    (instances
-      (project "schematic-main"
-        (path "/c9ad7189-d3b2-414a-9743-efd8e57cd755"
-          (reference "R23") (unit 1)
-        )
-        (path "/c9ad7189-d3b2-414a-9743-efd8e57cd755/f92f58ec-64e0-437c-bc00-8ae46a3b3054"
-          (reference "R38") (unit 1)
         )
       )
@@
         )
       )
-    )
-  )
-  (symbol (lib_id "Device:R") (at 141.351 122.174 180) (unit 1)
-    (in_bom yes) (on_board yes) (dnp no) (fields_autoplaced)
-    (property "Reference" "R23" (at 143.256 120.9039 0)
-      (effects (font (size 1.27 1.27)) (justify right))
-    )
-    (property "Value" "10k" (at 143.256 123.4439 0)
-      (effects (font (size 1.27 1.27)) (justify right))
-    )
-    (property "Footprint" "LED_SMD:LED_1206_3216Metric" (at 143.129 122.174 90)
-      (effects (font (size 1.27 1.27)) hide)
-    )
-    (property "Datasheet" "~" (at 141.351 122.174 0)
-      (effects (font (size 1.27 1.27)) hide)
-    )
-    (pin "1")
-    (pin "2")
-    (instances
-      (project "schematic-main"
-        (path "/c9ad7189-d3b2-414a-9743-efd8e57cd755"
-          (reference "R23") (unit 1)
-        )
-        (path "/c9ad7189-d3b2-414a-9743-efd8e57cd755/f92f58ec-64e0-437c-bc00-8ae46a3b3054"
-          (reference "R35") (unit 1)
-        )
-      )
-    )
-  )
-  (symbol (lib_id "Device:R") (at 135.382 141.224 180) (unit 1)
-    (in_bom yes) (on_board yes) (dnp no) (fields_autoplaced)
-    (property "Reference" "R23" (at 137.287 139.9539 0)
-      (effects (font (size 1.27 1.27)) (justify right))
-    )
-    (property "Value" "10k" (at 137.287 142.4939 0)
-      (effects (font (size 1.27 1.27)) (justify right))
-    )
-    (property "Footprint" "LED_SMD:LED_1206_3216Metric" (at 137.16 141.224 90)
-      (effects (font (size 1.27 1.27)) hide)
-    )
-    (property "Datasheet" "~" (at 135.382 141.224 0)
-      (effects (font (size 1.27 1.27)) hide)
-    )
-    (pin "1")
-    (pin "2")
-    (instances
-      (project "schematic-main"
-        (path "/c9ad7189-d3b2-414a-9743-efd8e57cd755"
-          (reference "R23") (unit 1)
-        )
-        (path "/c9ad7189-d3b2-414a-9743-efd8e57cd755/f92f58ec-64e0-437c-bc00-8ae46a3b3054"
-          (reference "R36") (unit 1)
-        )
-      )
