File: schematic-power.kicad_sch (KiCad schematic)
At the start: 35 parts, among them IC2 LM76202QPWPRQ1, U6 LM5013DDAR, U9 TPS62933

Commit message: Repair files
Parts:
- removed C26: 10u, Capacitor_SMD:CP_Elec_8x10.5, symbol Device:C_Polarized
- removed C27: 22u, Capacitor_SMD:CP_Elec_8x10.5, symbol Device:C_Polarized
- removed C28: 2n2, Capacitor_SMD:C_1206_3216Metric, symbol Device:C
- removed C29: 47p, Capacitor_SMD:C_1206_3216Metric, symbol Device:C
- removed C30: 3n3, Capacitor_SMD:C_1206_3216Metric, symbol Device:C
- removed D7: MBRD20100CT-13, MBRD20100CT-13:TO252_(DPAK)_1, symbol MBRD20100CT-13:MBRD20100CT-13
- removed F1, F2: 3A, mbr:FUSC8664X180N, symbol Device:Fuse
- removed L3: IHLP6767DZER470M11, library:IHLP6767DZER470M11, symbol IHLP6767DZER470M11:IHLP6767DZER470M11
- removed R14: 100k, Resistor_SMD:R_1206_3216Metric, symbol Device:R
- removed R15: 143k, Resistor_SMD:R_1206_3216Metric, symbol Device:R
- removed R24: 453k, LED_SMD:LED_1206_3216Metric, symbol Device:R
- removed R25: 49k9, LED_SMD:LED_1206_3216Metric, symbol Device:R
- removed U6: LM5013DDAR, Package_SO:Diodes_SO-8EP, symbol 2023-11-20_17-31-45:LM5013DDAR
Connections:
- no-connect marks 4 -> 3
Other:
- note removed: "Buck converter (+12 V)"

Commit message: P1
Parts:
- added C19 (x2): 100n, Capacitor_SMD:C_1206_3216Metric, symbol Device:C
- added C20: 10u, Capacitor_SMD:CP_Elec_8x10.5, symbol Device:C
- added PS1: TSR_1-2450, TSR-1-24120, symbol Tracko 1-2450 5V:TSR_1-2450
Connections:
- net GND: now also C19.2, C19.2, C20.2, PS1.2 (GND)
- net Vreg: now also C19.1, PS1.1 (VIN+)
- new net +5V: C19.1, C20.1, PS1.3 (VOUT+)
Other:
- note added: "Buck converter (+5 V)"
Changed lines of the file:
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@@
   (junction (at 77.6478 124.5616) (diameter 0) (color 0 0 0 0)
   )
+  (junction (at 228.6 53.34) (diameter 0) (color 0 0 0 0)
+  )
   (junction (at 232.41 141.5288) (diameter 0) (color 0 0 0 0)
   )
@@
   (junction (at 232.41 125.73) (diameter 0) (color 0 0 0 0)
   )
+  (junction (at 215.9 64.77) (diameter 0) (color 0 0 0 0)
+  )
   (junction (at 40.767 109.3216) (diameter 0) (color 0 0 0 0)
   )
+  (junction (at 203.2 64.77) (diameter 0) (color 0 0 0 0)
+  )
   (junction (at 62.357 118.2116) (diameter 0) (color 0 0 0 0)
   )
@@
   (junction (at 53.467 109.3216) (diameter 0) (color 0 0 0 0)
   )
+  (junction (at 215.9 53.34) (diameter 0) (color 0 0 0 0)
+  )
   (junction (at 248.92 133.35) (diameter 0) (color 0 0 0 0)
   )
@@
   )
   (junction (at 109.3724 106.7816) (diameter 0) (color 0 0 0 0)
+  )
+  (junction (at 190.5 53.34) (diameter 0) (color 0 0 0 0)
   )
   (junction (at 166.37 118.11) (diameter 0) (color 0 0 0 0)
@@
     (stroke (width 0) (type default))
   )
+  (wire (pts (xy 215.9 64.77) (xy 228.6 64.77))
+    (stroke (width 0) (type default))
+  )
   (wire (pts (xy 78.8924 119.4816) (xy 77.6224 119.4816))
     (stroke (width 0) (type default))
@@
     (stroke (width 0) (type default))
   )
+  (wire (pts (xy 190.5 64.77) (xy 203.2 64.77))
+    (stroke (width 0) (type default))
+  )
+  (wire (pts (xy 175.26 53.34) (xy 190.5 53.34))
+    (stroke (width 0) (type default))
+  )
   (wire (pts (xy 40.767 140.081) (xy 40.767 119.4816))
     (stroke (width 0) (type default))
   )
+  (wire (pts (xy 215.9 64.77) (xy 215.9 60.96))
+    (stroke (width 0) (type default))
+  )
   (wire (pts (xy 124.6886 140.4112) (xy 124.6886 134.0612))
     (stroke (width 0) (type default))
@@
     (stroke (width 0) (type default))
   )
+  (wire (pts (xy 240.665 53.34) (xy 228.6 53.34))
+    (stroke (width 0) (type default))
+  )
   (wire (pts (xy 113.7666 122.0724) (xy 113.7666 122.0216))
     (stroke (width 0) (type default))
@@
     (stroke (width 0) (type default))
   )
+  (wire (pts (xy 190.5 64.77) (xy 190.5 60.96))
+    (stroke (width 0) (type default))
+  )
   (wire (pts (xy 205.74 125.73) (xy 212.09 125.73))
     (stroke (width 0) (type default))
@@
     (stroke (width 0) (type default))
   )
+  (wire (pts (xy 215.9 53.34) (xy 228.6 53.34))
+    (stroke (width 0) (type default))
+  )
   (wire (pts (xy 124.6886 134.0612) (xy 124.6632 134.0612))
     (stroke (width 0) (type default))
@@
     (stroke (width 0) (type default))
   )
+  (wire (pts (xy 228.6 64.77) (xy 228.6 60.96))
+    (stroke (width 0) (type default))
+  )
   (wire (pts (xy 161.29 128.27) (xy 161.29 125.73))
     (stroke (width 0) (type default))
@@
   )
   (wire (pts (xy 77.6478 124.5616) (xy 77.6224 124.5616))
+    (stroke (width 0) (type default))
+  )
+  (wire (pts (xy 203.2 64.77) (xy 215.9 64.77))
     (stroke (width 0) (type default))
   )
@@
     (fill (type none))
   )
+  (rectangle (start 147.32 29.845) (end 267.335 84.455)
+    (stroke (width 0) (type dash))
+    (fill (type none))
+  )
   (text "C_{dVdt} = 47 x 10^{-6} / 8.7 x 10^{3} x 2 = 2.7 nF"
     (at 33.147 147.4216 0)
@@
     (effects (font (size 2 2)) (justify left bottom))
   )
+  (text "Buck converter (+5 V)" (at 147.32 29.21 0)
+    (effects (font (size 2 2)) (justify left bottom))
+  )
+  (label "Vreg" (at 175.26 53.34 0) (fields_autoplaced)
+    (effects (font (size 1.27 1.27)) (justify left bottom))
+  )
   (label "Vreg" (at 161.29 128.27 180) (fields_autoplaced)
     (effects (font (size 1.27 1.27)) (justify right bottom))
@@
     (effects (font (size 1.27 1.27)) (justify left))
   )
+  (hierarchical_label "+5V" (shape output) (at 240.665 53.34 0) (fields_autoplaced)
+    (effects (font (size 1.27 1.27)) (justify left))
+  )
   (hierarchical_label "VBUS" (shape input) (at 160.02 109.22 180) (fields_autoplaced)
     (effects (font (size 1.27 1.27)) (justify right))
@@
         (path "/c9ad7189-d3b2-414a-9743-efd8e57cd755/ed70203f-44bf-4bdc-8b45-a710eb8fc309"
           (reference "C1") (unit 1)
+        )
+      )
+    )
+  )
+  (symbol (lib_id "Tracko  1-2450 5V:TSR_1-2450") (at 190.5 52.07 0) (unit 1)
+    (in_bom yes) (on_board yes) (dnp no) (fields_autoplaced)
+    (property "Reference" "PS1" (at 203.2 45.085 0)
+      (effects (font (size 1.27 1.27)))
+    )
+    (property "Value" "TSR_1-2450" (at 203.2 47.625 0)
+      (effects (font (size 1.27 1.27)))
+    )
+    (property "Footprint" "TSR-1-24120" (at 212.09 146.99 0)
+      (effects (font (size 1.27 1.27)) (justify left top) hide)
+    )
+    (property "Datasheet" "https://tracopower.com/tsr1-datasheet/" (at 212.09 246.99 0)
+      (effects (font (size 1.27 1.27)) (justify left top) hide)
+    )
+    (property "Height" "" (at 212.09 446.99 0)
+      (effects (font (size 1.27 1.27)) (justify left top) hide)
+    )
+    (property "TME Electronic Components Part Number" "" (at 212.09 546.99 0)
+      (effects (font (size 1.27 1.27)) (justify left top) hide)
+    )
+    (property "TME Electronic Components Price/Stock" "" (at 212.09 646.99 0)
+      (effects (font (size 1.27 1.27)) (justify left top) hide)
+    )
+    (property "Manufacturer_Name" "Traco Power" (at 212.09 746.99 0)
+      (effects (font (size 1.27 1.27)) (justify left top) hide)
+    )
+    (property "Manufacturer_Part_Number" "TSR 1-2450" (at 212.09 846.99 0)
+      (effects (font (size 1.27 1.27)) (justify left top) hide)
+    )
+    (pin "1")
+    (pin "2")
+    (pin "3")
+    (instances
+      (project "schematic-main"
+        (path "/c9ad7189-d3b2-414a-9743-efd8e57cd755/ed70203f-44bf-4bdc-8b45-a710eb8fc309"
+          (reference "PS1") (unit 1)
         )
       )
@@
     )
   )
+  (symbol (lib_id "Device:C") (at 228.6 57.15 0) (unit 1)
+    (in_bom yes) (on_board yes) (dnp no) (fields_autoplaced)
+    (property "Reference" "C19" (at 231.775 55.88 0)
+      (effects (font (size 1.27 1.27)) (justify left))
+    )
+    (property "Value" "100n" (at 231.775 58.42 0)
+      (effects (font (size 1.27 1.27)) (justify left))
+    )
+    (property "Footprint" "Capacitor_SMD:C_1206_3216Metric" (at 229.5652 60.96 0)
+      (effects (font (size 1.27 1.27)) hide)
+    )
+    (property "Datasheet" "~" (at 228.6 57.15 0)
+      (effects (font (size 1.27 1.27)) hide)
+    )
+    (pin "1")
+    (pin "2")
+    (instances
+      (project "schematic-power"
+        (path "/6159aad4-3df8-4b77-bdff-c4df127c8492"
+          (reference "C19") (unit 1)
+        )
+      )
+      (project "schematic-main"
+        (path "/c9ad7189-d3b2-414a-9743-efd8e57cd755/ed70203f-44bf-4bdc-8b45-a710eb8fc309"
+          (reference "C28") (unit 1)
+        )
+      )
+    )
+  )
   (symbol (lib_id "Device:R") (at 232.41 129.54 0) (unit 1)
     (in_bom yes) (on_board yes) (dnp no) (fields_autoplaced)
@@
     )
   )
+  (symbol (lib_id "power:GND") (at 203.2 64.77 0) (unit 1)
+    (in_bom yes) (on_board yes) (dnp no) (fields_autoplaced)
+    (property "Reference" "#PWR035" (at 203.2 71.12 0)
+      (effects (font (size 1.27 1.27)) hide)
+    )
+    (property "Value" "GND" (at 203.2 69.215 0)
+      (effects (font (size 1.27 1.27)) hide)
+    )
+    (property "Footprint" "" (at 203.2 64.77 0)
+      (effects (font (size 1.27 1.27)) hide)
+    )
+    (property "Datasheet" "" (at 203.2 64.77 0)
+      (effects (font (size 1.27 1.27)) hide)
+    )
+    (pin "1")
+    (instances
+      (project "schematic-power"
+        (path "/6159aad4-3df8-4b77-bdff-c4df127c8492"
+          (reference "#PWR035") (unit 1)
+        )
+      )
+      (project "schematic-main"
+        (path "/c9ad7189-d3b2-414a-9743-efd8e57cd755/ed70203f-44bf-4bdc-8b45-a710eb8fc309"
+          (reference "#PWR053") (unit 1)
+        )
+      )
+    )
+  )
   (symbol (lib_id "power:GND") (at 195.58 138.43 0) (unit 1)
     (in_bom yes) (on_board yes) (dnp no) (fields_autoplaced)
@@
         (path "/c9ad7189-d3b2-414a-9743-efd8e57cd755/ed70203f-44bf-4bdc-8b45-a710eb8fc309"
           (reference "#PWR07") (unit 1)
+        )
+      )
+    )
+  )
+  (symbol (lib_id "Device:C") (at 215.9 57.15 0) (unit 1)
+    (in_bom yes) (on_board yes) (dnp no)
+    (property "Reference" "C20" (at 219.075 55.8799 0)
+      (effects (font (size 1.27 1.27)) (justify left))
+    )
+    (property "Value" "10u" (at 219.075 58.4199 0)
+      (effects (font (size 1.27 1.27)) (justify left))
+    )
+    (property "Footprint" "Capacitor_SMD:CP_Elec_8x10.5" (at 216.8652 60.96 0)
+      (effects (font (size 1.27 1.27)) hide)
+    )
+    (property "Datasheet" "~" (at 215.9 57.15 0)
+      (effects (font (size 1.27 1.27)) hide)
+    )
+    (pin "1")
+    (pin "2")
+    (instances
+      (project "schematic-power"
+        (path "/6159aad4-3df8-4b77-bdff-c4df127c8492"
+          (reference "C20") (unit 1)
+        )
+      )
+      (project "schematic-main"
+        (path "/c9ad7189-d3b2-414a-9743-efd8e57cd755/ed70203f-44bf-4bdc-8b45-a710eb8fc309"
+          (reference "C27") (unit 1)
         )
       )
@@
         )
       )
+    )
+  )
+  (symbol (lib_id "Device:C") (at 190.5 57.15 0) (mirror y) (unit 1)
+    (in_bom yes) (on_board yes) (dnp no)
+    (property "Reference" "C19" (at 187.325 55.88 0)
+      (effects (font (size 1.27 1.27)) (justify left))
+    )
+    (property "Value" "100n" (at 187.325 58.42 0)
+      (effects (font (size 1.27 1.27)) (justify left))
+    )
+    (property "Footprint" "Capacitor_SMD:C_1206_3216Metric" (at 189.5348 60.96 0)
+      (effects (font (size 1.27 1.27)) hide)
+    )
+    (property "Datasheet" "~" (at 190.5 57.15 0)
+      (effects (font (size 1.27 1.27)) hide)
+    )
+    (pin "1")
+    (pin "2")
+    (instances
+      (project "schematic-power"
+        (path "/6159aad4-3df8-4b77-bdff-c4df127c8492"
+          (reference "C19") (unit 1)
+        )
+      )
+      (project "schematic-main"
+        (path "/c9ad7189-d3b2-414a-9743-efd8e57cd755/ed70203f-44bf-4bdc-8b45-a710eb8fc309"
+          (reference "C29") (unit 1)
+        )
+      )
