File: schematic-main.kicad_pcb (KiCad board)
At the start: 2 copper layers, 100 x 100 mm, 65 parts, among them IC1 LM76202QPWPRQ1, IC2 AD8544ARUZ-REEL, IC3 ACHS-7123-000E, IC4 ACHS-7121-000E, IC5 ACHS-7123-000E, IC6 LM5106MMX_NOPB, IC7 LM5106MMX_NOPB, J1 Battery converter, J2 CAN, J3 FUEL CELL, J4 Joulemeter, J5 MOTOR CONTROLER, J6 SUPER CAPACITORS, P1 USB_C_Plug_USB2.0, Q1 CSD19531Q5AT, Q2 CSD19531Q5AT, Q3 CSD19531Q5AT, Q4 CSD19531Q5AT, U1 TPS62933, U2 USBLC6-2P6, U4 ESP32-S3FN8, Y1 Crystal_GND24

Commit message: PCB design 50%
Parts:
- added C1: 1u, Capacitor_SMD:C_1206_3216Metric, F.Cu at (206.4, 68.1)
- added C10: 47p, Capacitor_SMD:C_1206_3216Metric, F.Cu at (206.4, 88.2)
- added C11: 100n, Capacitor_SMD:C_1206_3216Metric, F.Cu at (206.4, 91.5)
- added C12: 100u, Capacitor_SMD:CP_Elec_8x10.5, F.Cu at (131.1, 39.1)
- added C13: 1u, Capacitor_SMD:C_1206_3216Metric, F.Cu at (90.1, 114.2)
- added C16: 100n, Capacitor_SMD:C_1206_3216Metric, F.Cu at (105.5, 136.5)
- added C17: 1u, Capacitor_SMD:C_1206_3216Metric, F.Cu at (90.1, 119.6)
- added C18: 1u, Capacitor_SMD:C_1206_3216Metric, F.Cu at (90.2, 124.6)
- added C2: 47u, Capacitor_SMD:CP_Elec_6.3x7.7, F.Cu at (97.6, 42.1)
- added C25: 1u, Capacitor_SMD:C_1206_3216Metric, F.Cu at (98.2, 106.8)
- added C27: 4n7, Capacitor_SMD:C_1206_3216Metric, F.Cu at (72.1, 72.9)
- added C28: 100n, Capacitor_SMD:C_1206_3216Metric, F.Cu at (73.5, 78.6)
- added C29: 4n7, Capacitor_SMD:C_1206_3216Metric, F.Cu at (73.8, 82.9)
- added C3: 2n7, Capacitor_SMD:C_1206_3216Metric, F.Cu at (206.4, 71.5)
- added C30: 4n7, Capacitor_SMD:C_1206_3216Metric, F.Cu at (103.0, 85.0)
- added C31: 100n, Capacitor_SMD:C_1206_3216Metric, F.Cu at (74.0, 93.7)
- added C33: 100n, Capacitor_SMD:C_1206_3216Metric, F.Cu at (196.2, 126.6)
- added C34: 1n, Capacitor_SMD:C_1206_3216Metric, F.Cu at (161.4, 115.4)
- added C35: 100n, Capacitor_SMD:C_1206_3216Metric, F.Cu at (66.3, 116.0)
- added C36: 1n, Capacitor_SMD:C_1206_3216Metric, F.Cu at (151.8, 125.6)
- added C37: 100n, Capacitor_SMD:C_1206_3216Metric, F.Cu at (66.3, 122.7)
- added C38: 1n, Capacitor_SMD:C_1206_3216Metric, F.Cu at (173.2, 119.8)
- added C39: 1n, Capacitor_SMD:C_1206_3216Metric, F.Cu at (76.8, 144.2)
- added C4: 10u, Capacitor_SMD:CP_Elec_8x10.5, F.Cu at (111.0, 39.1)
- added C40: 470n, Capacitor_SMD:C_1206_3216Metric, F.Cu at (76.8, 147.6)
- added C41: 10n, Capacitor_SMD:C_1206_3216Metric, F.Cu at (76.8, 150.9)
- added C42: 100n 100V, Capacitor_SMD:C_1206_3216Metric, F.Cu at (129.2, 77.0)
- added C43: 100p 100V, Capacitor_SMD:C_1206_3216Metric, F.Cu at (76.8, 157.6)
- added C44: 100p 100V, Capacitor_SMD:C_1206_3216Metric, F.Cu at (76.8, 160.9)
- added C46: 1n, Capacitor_SMD:C_1206_3216Metric, F.Cu at (68.0, 131.8)
- added C47: 470n, Capacitor_SMD:C_1206_3216Metric, F.Cu at (68.0, 135.2)
- added C48: 10n, Capacitor_SMD:C_1206_3216Metric, F.Cu at (68.0, 138.6)
- added C49: 100n 100V, Capacitor_SMD:C_1206_3216Metric, F.Cu at (68.0, 141.9)
- added C5: 33n, Capacitor_SMD:C_1206_3216Metric, F.Cu at (206.4, 74.8)
- added C50: 100n, Capacitor_SMD:C_1206_3216Metric, F.Cu at (100.0, 135.5)
- added C6: 100n, Capacitor_SMD:C_1206_3216Metric, F.Cu at (206.4, 78.2)
- added C7: 100n, Capacitor_SMD:C_1206_3216Metric, F.Cu at (206.4, 81.5)
- added C8: 100n, Capacitor_SMD:C_1206_3216Metric, F.Cu at (206.4, 84.8)
- added C9: 10u, Capacitor_SMD:CP_Elec_8x10.5, F.Cu at (121.0, 39.1)
- added D10: SKL120-AQ, Lib:SODFL3718X170N, F.Cu at (195.4, 106.7)
- added D11: SKL120-AQ, Lib:SODFL3718X170N, F.Cu at (195.4, 110.0)
- added D12: SKL120-AQ, Lib:SODFL3718X170N, F.Cu at (195.4, 113.4)
- added D3: SP0502BAJT, Package_TO_SOT_SMD:SOT-323_SC-70, F.Cu at (104.3, 91.2)
- added D6: LED, Diode_SMD:D_1206_3216Metric, F.Cu at (84.4, 44.8)
- added D7: SKL120-AQ, Lib:SODFL3718X170N, F.Cu at (148.8, 68.0)
- added D8: SKL120-AQ, Lib:SODFL3718X170N, F.Cu at (195.4, 100.0)
- added D9: SKL120-AQ, Lib:SODFL3718X170N, F.Cu at (141.0, 75.6)
- added IC8: MCP4018T-503E_LT, Lib:SOT65P210X110-6N, F.Cu at (96.5, 134.0)
- added JP1: SolderJumper_2_Open, Jumper:SolderJumper-2_P1.3mm_Open_Pad1.0x1.5mm, F.Cu at (87.7, 114.2)
- added JP2: SolderJumper_2_Open, Jumper:SolderJumper-2_P1.3mm_Open_Pad1.0x1.5mm, F.Cu at (87.7, 119.8)
- added JP3: SolderJumper_2_Open, Jumper:SolderJumper-2_P1.3mm_Open_Pad1.0x1.5mm, F.Cu at (87.8, 124.6)
- added R10: 32k, Resistor_SMD:R_1206_3216Metric, F.Cu at (203.6, 57.5)
- added R11: 10k, Resistor_SMD:R_1206_3216Metric, F.Cu at (203.6, 60.8)
- added R12: 10k, Resistor_SMD:R_1206_3216Metric, F.Cu at (92.7, 116.4)
- added R13: 10k, Resistor_SMD:R_1206_3216Metric, F.Cu at (93.9, 120.2)
- added R14: 10k, LED_SMD:LED_1206_3216Metric, F.Cu at (93.0, 124.4)
- added R15: 60, Resistor_SMD:R_1206_3216Metric, F.Cu at (107.0, 88.0)
- added R16: 60, LED_SMD:LED_1206_3216Metric, F.Cu at (107.0, 85.0)
- added R19: 1k, LED_SMD:LED_1206_3216Metric, F.Cu at (84.4, 47.4)
- added R26: 10k, LED_SMD:LED_1206_3216Metric, F.Cu at (165.2, 116.8)
- added R27: 20k, LED_SMD:LED_1206_3216Metric, F.Cu at (161.4, 118.2)
- added R28: 10k, LED_SMD:LED_1206_3216Metric, F.Cu at (153.2, 121.8)
- added R29: 20k, LED_SMD:LED_1206_3216Metric, F.Cu at (154.6, 125.6)
- added R30: 10k, LED_SMD:LED_1206_3216Metric, F.Cu at (169.4, 118.6)
- added R31: 20k, LED_SMD:LED_1206_3216Metric, F.Cu at (173.2, 117.0)
- added R32: 68k, LED_SMD:LED_1206_3216Metric, F.Cu at (19.2, 51.6)
- added R33: 3k9, LED_SMD:LED_1206_3216Metric, F.Cu at (19.2, 55.0)
- added R34: 10R 2W, LED_SMD:LED_1206_3216Metric, F.Cu at (148.8, 71.2)
- added R35: 100R 0,5W, LED_SMD:LED_1206_3216Metric, F.Cu at (24.9, 34.6)
- added R36: 100R 0,5W, LED_SMD:LED_1206_3216Metric, F.Cu at (24.9, 38.0)
- added R37: 10k, LED_SMD:LED_1206_3216Metric, F.Cu at (24.9, 41.4)
- added R38: 10R 2W, LED_SMD:LED_1206_3216Metric, F.Cu at (24.9, 44.8)
- added R39: 200R, LED_SMD:LED_1206_3216Metric, F.Cu at (24.9, 48.2)
- added R40: 200R, LED_SMD:LED_1206_3216Metric, F.Cu at (24.9, 51.6)
- added R41: 62k, LED_SMD:LED_1206_3216Metric, F.Cu at (24.9, 55.0)
- added R42: 4k7, LED_SMD:LED_1206_3216Metric, F.Cu at (64.8, 26.7)
- added R43: 10k, LED_SMD:LED_1206_3216Metric, F.Cu at (89.8, 128.4)
- added R44: 10k, LED_SMD:LED_1206_3216Metric, F.Cu at (91.6, 131.2)
- added R45: 10R 2W, LED_SMD:LED_1206_3216Metric, F.Cu at (68.2, 26.7)
- added R5: 180k, Resistor_SMD:R_1206_3216Metric, F.Cu at (203.6, 41.0)
- added R50: 0R, LED_SMD:LED_1206_3216Metric, F.Cu at (78.4, 26.7)
- added R51: 0R, LED_SMD:LED_1206_3216Metric, F.Cu at (81.8, 26.7)
- added R52: 10k, LED_SMD:LED_1206_3216Metric, F.Cu at (91.6, 134.6)
- added R53: 10k, LED_SMD:LED_1206_3216Metric, F.Cu at (91.5, 137.5)
- added R54: 4,7k, LED_SMD:LED_1206_3216Metric, F.Cu at (111.4, 130.6)
- added R55: 4,7k, LED_SMD:LED_1206_3216Metric, F.Cu at (115.8, 129.6)
- added R6: 12k, Resistor_SMD:R_1206_3216Metric, F.Cu at (203.6, 44.3)
- added R7: 100k, Resistor_SMD:R_1206_3216Metric, F.Cu at (203.6, 47.6)
- added R8: 100k, Resistor_SMD:R_1206_3216Metric, F.Cu at (203.6, 50.9)
- added R9: 56k, Resistor_SMD:R_1206_3216Metric, F.Cu at (203.6, 54.2)
- added TP13: FC test, Connector_PinSocket_2.54mm:PinSocket_1x01_P2.54mm_Vertical, F.Cu at (118.8, 135.2)
- added TP14: FC_C_test, Connector_PinSocket_2.54mm:PinSocket_1x01_P2.54mm_Vertical, F.Cu at (157.6, 123.6)
- added TP15: SC_C_test, Connector_PinSocket_2.54mm:PinSocket_1x01_P2.54mm_Vertical, F.Cu at (164.4, 121.4)
- added TP16: MC_C_test, Connector_PinSocket_2.54mm:PinSocket_1x01_P2.54mm_Vertical, F.Cu at (169.8, 114.0)
- added TP17: EN test, Connector_PinSocket_2.54mm:PinSocket_1x01_P2.54mm_Vertical, F.Cu at (44.4, 89.8)
- added TP18: PWM test, Connector_PinSocket_2.54mm:PinSocket_1x01_P2.54mm_Vertical, F.Cu at (44.6, 82.2)
- added TP19: SC test, Connector_PinSocket_2.54mm:PinSocket_1x01_P2.54mm_Vertical, F.Cu at (46.8, 46.6)
- added TP21: EN test, Connector_PinSocket_2.54mm:PinSocket_1x01_P2.54mm_Vertical, F.Cu at (46.8, 51.2)
- added TP22: PWM test, Connector_PinSocket_2.54mm:PinSocket_1x01_P2.54mm_Vertical, F.Cu at (46.8, 55.8)
- added TP23: D_Pot_W, Connector_PinSocket_2.54mm:PinSocket_1x01_P2.54mm_Vertical, F.Cu at (87.0, 131.6)
- added TP24: D_Pot_A, Connector_PinSocket_2.54mm:PinSocket_1x01_P2.54mm_Vertical, F.Cu at (87.0, 136.6)
- added TP3: +12V, Connector_PinSocket_2.54mm:PinSocket_1x01_P2.54mm_Vertical, F.Cu at (62.7, 55.2)
- added TP4: +12V, Connector_PinSocket_2.54mm:PinSocket_1x01_P2.54mm_Vertical, F.Cu at (62.7, 59.8)
- added TP5: +5V, Connector_PinSocket_2.54mm:PinSocket_1x01_P2.54mm_Vertical, F.Cu at (71.2, 60.2)
- added TP6: +5V, Connector_PinSocket_2.54mm:PinSocket_1x01_P2.54mm_Vertical, F.Cu at (71.2, 64.8)
- added TP7: +3.3V, Connector_PinSocket_2.54mm:PinSocket_1x01_P2.54mm_Vertical, F.Cu at (79.6, 56.6)
- added TP8: +3.3V, Connector_PinSocket_2.54mm:PinSocket_1x01_P2.54mm_Vertical, F.Cu at (79.6, 61.2)
- added U4: SN65HVD232, Package_SO:SOIC-8_3.9x4.9mm_P1.27mm, F.Cu at (114.0, 86.3)
- C19: renamed from C28; value 10n -> 10u; footprint Capacitor_SMD:C_1206_3216Metric -> Capacitor_SMD:CP_Elec_8x10.5
- C21: renamed from C27; value 1u -> 100n
- C26: renamed from C23; value 100n -> 10n
- D4: renamed from D5; footprint LED_SMD:LED_1206_3216Metric -> Diode_SMD:D_1206_3216Metric
- D5: renamed from D6; footprint LED_SMD:LED_1206_3216Metric -> Diode_SMD:D_1206_3216Metric
- J2: footprint library:39303035 -> Lib:39303035
- L3: moved to F.Cu
- R17: renamed from R35; footprint Resistor_SMD:R_1206_3216Metric -> LED_SMD:LED_1206_3216Metric
- R18: renamed from R36; footprint Resistor_SMD:R_1206_3216Metric -> LED_SMD:LED_1206_3216Metric
- R24: renamed from R29; footprint Resistor_SMD:R_1206_3216Metric -> LED_SMD:LED_1206_3216Metric
- R25: renamed from R30; footprint Resistor_SMD:R_1206_3216Metric -> LED_SMD:LED_1206_3216Metric
- R47: value 10k -> 10R 2W; footprint Resistor_SMD:R_1206_3216Metric -> LED_SMD:LED_1206_3216Metric
- R48: value 10k -> 200R; footprint Resistor_SMD:R_1206_3216Metric -> LED_SMD:LED_1206_3216Metric
- moved R48 141.4 mm to (75.0, 26.7), turned to 90 degrees
- moved R47 140.2 mm to (71.6, 26.7), turned to 90 degrees
- moved R21 93.5 mm to (101.4, 122.8)
- moved TP12 93.3 mm to (101.2, 128.4)
- moved R20 92.2 mm to (100.0, 120.2)
- moved R25 91.7 mm to (110.4, 128.0)
- moved C20 91.7 mm to (100.7, 106.8)
- moved C21 91.7 mm to (103.2, 106.8)
- moved C26 91.7 mm to (100.5, 111.8)
- moved D5 91.7 mm to (124.8, 116.2)
- moved R23 91.7 mm to (105.6, 128.2)
- moved TP1 91.7 mm to (89.0, 102.2)
- moved TP2 91.7 mm to (94.0, 102.2)
- moved U3 91.7 mm to (112.3, 115.2)
- moved C14 91.7 mm to (107.5, 108.1)
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- renumbered C17 to C14, C16 to C15, C22 to C20, C24 to C22, C25 to C23, C26 to C24, L3 to L2, R25 to R20, R26 to R21, R27 to R22, R28 to R23, TP2 to TP1, TP2 to TP10, TP12 to TP11, TP13 to TP12, TP3 to TP2, TP1 to TP9, U4 to U3
Connections:
- C14 pad 1: /MCU/XTAL_P -> /MCU/XTAL_N
- C15 pad 1: /MCU/XTAL_N -> /MCU/XTAL_P
- C45 pad 1: /Converter/SC_c2 -> /Converter/SC_c1
- F2 pad 1: /Converter/MC_c2 -> /Converter/MC_c1
- F2 pad 2: /Converter/SC_c1 -> /Converter/SC_c2
- J4 pad 1: /Converter/MC_c2 -> /Converter/MC_c1
- J5 pad 1: /Converter/MC_c1 -> /Converter/MC_c2
- J6 pad 1: /Converter/MC_c2 -> /Converter/MC_c1
- Q4 pad 5: /Converter/SC_c2 -> /Converter/SC_c1
- Q4 pad 6: /Converter/SC_c2 -> /Converter/SC_c1
- Q4 pad 7: /Converter/SC_c2 -> /Converter/SC_c1
- Q4 pad 8: /Converter/SC_c2 -> /Converter/SC_c1
- Q4 pad 9: /Converter/SC_c2 -> /Converter/SC_c1
- R20 pad 1: (no net) -> Net-(R20-Pad1)
- R21 pad 1: (no net) -> Net-(R21-Pad1)
- R22 pad 1: (no net) -> Net-(R22-Pad1)
- R23 pad 1: (no net) -> Net-(R23-Pad1)
- R47 pad 1: (no net) -> /Converter/Low_mosfet_B
- R47 pad 2: GND -> Net-(D12-A)
- R48 pad 1: (no net) -> /Converter/Converter_ON_B_MCU
- R48 pad 2: +3.3V -> Net-(IC7-EN)
- TP10 pad 1: (no net) -> Net-(R21-Pad1)
- TP11 pad 1: (no net) -> Net-(R22-Pad1)
- TP12 pad 1: (no net) -> Net-(R23-Pad1)
- TP9 pad 1: (no net) -> Net-(R20-Pad1)
- U3 pad 1: (no net) -> unconnected-(U3-LNA_IN/RF-Pad1)
- U3 pad 10: (no net) -> /IO/FC_Voltage_MCU
- U3 pad 11: (no net) -> unconnected-(U3-GPIO6/ADC1_CH5-Pad11)
- U3 pad 14: (no net) -> /Converter/FC_c_MCU
- U3 pad 15: (no net) -> unconnected-(U3-GPIO10/ADC1_CH9-Pad15)
- U3 pad 17: (no net) -> unconnected-(U3-GPIO12/ADC2_CH1-Pad17)
- U3 pad 19: (no net) -> unconnected-(U3-GPIO14/ADC2_CH3-Pad19)
- U3 pad 21: (no net) -> unconnected-(U3-GPIO15/ADC2_CH4/XTAL_32K_P-Pad21)
- U3 pad 22: (no net) -> unconnected-(U3-GPIO16/ADC2_CH5/XTAL_32K_N-Pad22)
- U3 pad 23: (no net) -> /Converter/SC_c_MCU
- U3 pad 24: (no net) -> /Converter/MC_c_MCU
- U3 pad 27: (no net) -> /IO/SDA_D_Pot_i2c_MCU
- U3 pad 28: (no net) -> /IO/SCL_D_Pot_i2c_MCU
- U3 pad 29: (no net) -> unconnected-(U3-VDD_SPI-Pad29)
- U3 pad 30: (no net) -> /MCU/Converter_PWM_A_MCU
- U3 pad 31: (no net) -> /MCU/Converter_ON_A_MCU
- U3 pad 32: (no net) -> unconnected-(U3-SPICS0/GPIO29-Pad32)
- U3 pad 33: (no net) -> unconnected-(U3-SPICLK/GPIO30-Pad33)
- U3 pad 34: (no net) -> unconnected-(U3-SPIQ/GPIO31-Pad34)
- U3 pad 36: (no net) -> unconnected-(U3-SPICLK_N/GPIO48-Pad36)
- U3 pad 37: (no net) -> unconnected-(U3-SPICLK_P/GPIO47-Pad37)
- U3 pad 39: (no net) -> unconnected-(U3-GPIO34-Pad39)
- U3 pad 40: (no net) -> unconnected-(U3-GPIO35-Pad40)
- U3 pad 41: (no net) -> /Converter/Converter_PWM_B_MCU
- U3 pad 42: (no net) -> /Converter/Converter_ON_B_MCU
- U3 pad 43: (no net) -> unconnected-(U3-GPIO38-Pad43)
- U3 pad 47: (no net) -> unconnected-(U3-MTDI/JTAG/GPIO41-Pad47)
- U3 pad 48: (no net) -> unconnected-(U3-MTMS/JTAG/GPIO42-Pad48)
- U3 pad 49: (no net) -> unconnected-(U3-U0TXD/PROG/GPIO43-Pad49)
- U3 pad 50: (no net) -> unconnected-(U3-U0RXD/PROG/GPIO44-Pad50)
- U3 pad 51: (no net) -> unconnected-(U3-GPIO45-Pad51)
- U3 pad 52: (no net) -> unconnected-(U3-GPIO46-Pad52)
- U3 pad 7: (no net) -> unconnected-(U3-GPIO2/ADC1_CH1-Pad7)
- U3 pad 8: (no net) -> /IO/SC_Voltage_MCU
- U3 pad 9: /IO/FC_Voltage_MCU -> unconnected-(U3-GPIO4/ADC1_CH3-Pad9)
Routing:
- net GND: track 185.9 -> 428.5 mm, vias 21 -> 48
- net (no net): track 133.4 -> 0.00 mm, vias 11 -> 0
- net /Converter/FC_c_MCU: track 0.00 -> 74.0 mm, vias 0 -> 1
- net /Converter/MC_c_MCU: track 0.00 -> 72.1 mm, vias 0 -> 1
- net /Converter/SC_c_MCU: track 0.00 -> 66.4 mm, vias 0 -> 1
- net /Converter/MC_c2: track 90.6 -> 25.7 mm
- net +3.3V: track 102.9 -> 164.1 mm, vias 5 -> 7
- net /Converter/Bootstrap_A: track 0.00 -> 57.0 mm
- net /Converter/Bootstrap_B: track 0.00 -> 55.8 mm
- net /IO/SCL_D_Pot_i2c_MCU: track 0.00 -> 37.8 mm, vias 0 -> 2
- net /Converter/FC_c2: track 13.8 -> 48.8 mm
- net /Converter/SC_c2: track 53.5 -> 19.4 mm
- net +5V: track 0.00 -> 33.3 mm
- net /IO/SDA_D_Pot_i2c_MCU: track 0.00 -> 33.3 mm, vias 0 -> 2
- net /Converter/MC_c1: track 50.8 -> 19.3 mm
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
Commit message: PCB design 80%
Parts:
- added REF**: MountingHole_3.2mm_M3, MountingHole:MountingHole_3.2mm_M3, F.Cu at (179.6, 105.6)
- added REF**: MountingHole_3.2mm_M3, MountingHole:MountingHole_3.2mm_M3, F.Cu at (90.6, 144.4)
- added REF**: MountingHole_3.2mm_M3, MountingHole:MountingHole_3.2mm_M3, F.Cu at (179.6, 55.4)
- added REF**: MountingHole_3.2mm_M3, MountingHole:MountingHole_3.2mm_M3, F.Cu at (90.6, 55.6)
- moved C44 182.0 mm to (188.3, 17.2), turned to 90 degrees
- moved C43 177.3 mm to (185.0, 17.2), turned to 90 degrees
- moved C41 167.9 mm to (178.3, 17.2), turned to 90 degrees
- moved TP19 167.2 mm to (191.2, 130.8)
- moved C40 163.2 mm to (174.9, 17.2), turned to 90 degrees
- moved C39 158.5 mm to (171.6, 17.2), turned to 90 degrees
- moved C49 153.9 mm to (169.3, 26.0), turned to 90 degrees
- moved C48 149.2 mm to (165.9, 26.0), turned to 90 degrees
- moved C47 144.5 mm to (162.6, 26.0), turned to 90 degrees
- moved C37 126.7 mm to (150.1, 27.6), turned to 90 degrees
- moved C35 117.2 mm to (143.4, 27.6), turned to 90 degrees
- moved R41 112.3 mm to (127.6, 100.4)
- moved R51 111.0 mm to (163.4, 102.0), turned to 180 degrees
- moved R32 105.1 mm to (113.4, 98.2), turned to 90 degrees
- moved R42 102.3 mm to (128.4, 106.8)
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Connections:
- C1 pad 1: /VBUS -> /Power /Vin
- D1 pad 2: /VBUS -> /Power /Vin
- IC1 pad 1: /VBUS -> /Power /Vin
- IC1 pad 2: /VBUS -> /Power /Vin
- IC1 pad 3: /VBUS -> /Power /Vin
- J1 pad 2: /Vin -> /Power /Vin
- R5 pad 1: /VBUS -> /Power /Vin
Routing:
- net GND: track 428.5 -> 860.2 mm, vias 48 -> 55
- net +5V: track 33.3 -> 187.7 mm, vias 0 -> 1
- net +3.3V: track 164.1 -> 270.6 mm, vias 7 -> 9
- net /VBUS: track 38.6 -> 112.2 mm
- net /Converter/MC_c1: track 19.3 -> 78.3 mm
- net /Converter/Converter_PWM_B_MCU: track 0.00 -> 50.0 mm, vias 0 -> 1
- net /MCU/Converter_PWM_A_MCU: track 9.92 -> 50.8 mm, vias 1 -> 0
- net /Converter/Converter_ON_B_MCU: track 9.51 -> 48.9 mm, vias 2 -> 1
- net /Converter/Low_mosfet_A: track 1.34 -> 38.2 mm, vias 1 -> 3
- net /MCU/Converter_ON_A_MCU: track 10.4 -> 46.9 mm, vias 1 -> 0
- net /Converter/FC_c2: track 48.8 -> 85.3 mm, vias 0 -> 2
- net /Converter/SC_c1: track 31.4 -> 65.7 mm, vias 0 -> 2
- net /Converter/Bootstrap_B: track 55.8 -> 89.1 mm
- net /Converter/Low_mosfet_B: track 1.42 -> 34.0 mm
- net /Converter/Bootstrap_A: track 57.0 -> 82.0 mm
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
Commit message: PCB design complate
Parts:
- (R50): renamed from R50; footprint LED_SMD:LED_1206_3216Metric -> Resistor_SMD:R_2512_6332Metric_Pad1.40x3.35mm_HandSolder
- C43, C44: moved to B.Cu
- R14, R16, R17, R18, R19, R24, R25, R26, R27, R28, R29, R30, R31, R32, R33, R37, R39, R40, R41, R42, R43, R44, R46, R48, R49, R52, R53, R54, R55: footprint LED_SMD:LED_1206_3216Metric -> Resistor_SMD:R_1206_3216Metric
- R34, R38, R45, R47: footprint LED_SMD:LED_1206_3216Metric -> Resistor_SMD:R_2512_6332Metric
- R35, R36: footprint LED_SMD:LED_1206_3216Metric -> Resistor_SMD:R_2512_6332Metric; moved to B.Cu
- R51: footprint LED_SMD:LED_1206_3216Metric -> Resistor_SMD:R_2512_6332Metric_Pad1.40x3.35mm_HandSolder
- TP17: value EN test -> EN A test
- TP18: value PWM test -> PWM A test
- TP21: value EN test -> EN B test
- TP22: value PWM test -> PWM B test
- moved R35 180.7 mm to (199.2, 82.2), turned to 90 degrees
- moved R36 152.0 mm to (169.0, 86.3), turned to -90 degrees
- moved R40 113.3 mm to (130.9, 91.4), turned to -90 degrees
- moved R39 110.7 mm to (127.3, 90.2), turned to 180 degrees
- moved R37 108.0 mm to (130.1, 65.9)
- moved R38 105.4 mm to (127.3, 69.6)
- moved C39 102.6 mm to (111.0, 100.0), turned to 180 degrees
- moved C35 97.2 mm to (166.6, 122.0), turned to -90 degrees
- moved R9 95.6 mm to (114.9, 62.0)
- moved R6 94.9 mm to (114.0, 76.2)
- moved R8 92.9 mm to (109.6, 62.4)
- moved R7 92.6 mm to (117.7, 67.6)
- moved C3 92.3 mm to (114.3, 64.7)
- moved C37 91.6 mm to (157.5, 119.0)
- moved R45 90.0 mm to (143.3, 76.4), turned to 0 degrees
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- renumbered C15 to C14, C14 to C15
Connections:
- R39 pad 1: /Converter/Converter_ON_B_MCU -> /Converter/Converter_ON_A_MCU
- R40 pad 2: /Converter/Converter_PWM_B_MCU -> /Converter/Converter_PWM_A_MCU
- U3 pad 30: /MCU/Converter_PWM_A_MCU -> /Converter/Converter_PWM_A_MCU
- U3 pad 31: /MCU/Converter_ON_A_MCU -> /Converter/Converter_ON_A_MCU
Routing:
- net GND: track 860.2 -> 1052.6 mm, vias 55 -> 229
- net +3.3V: track 270.6 -> 387.8 mm, vias 9 -> 15
- net +12V: track 0.00 -> 95.0 mm, vias 0 -> 1
- net +5V: track 187.7 -> 270.7 mm
- net Net-(U1-VIN): track 0.00 -> 56.0 mm
- net /Converter/Converter_ON_A_MCU: track 0.00 -> 51.4 mm
- net /Converter/Converter_PWM_A_MCU: track 0.00 -> 51.0 mm
- net /MCU/Converter_PWM_A_MCU: track 50.8 -> 0.00 mm
- net /Converter/Bootstrap_B: track 89.1 -> 139.3 mm, vias 0 -> 2
- net /Converter/Bootstrap_A: track 82.0 -> 131.9 mm
- net /MCU/Converter_ON_A_MCU: track 46.9 -> 0.00 mm
- net /Converter/Low_mosfet_A: track 38.2 -> 73.5 mm, vias 3 -> 4
- net /Power /Vin: track 11.1 -> 42.3 mm
- net Net-(IC6-EN): track 0.00 -> 30.6 mm, vias 0 -> 1
- net Net-(IC6-IN): track 0.00 -> 29.7 mm, vias 0 -> 1
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- added copper zone on B.Cu, net +12V
- added copper zone on F.Cu, net +12V
- added copper zone on F.Cu, net +3.3V
- added copper zone on F.Cu, net +5V
- added copper zone on F.Cu, net /Converter/FC_c1
- added copper zone on F.Cu, net /Converter/FC_c2
- added copper zone on F.Cu, net /Converter/MC_c1
- added copper zone on F.Cu, net /Converter/MC_c2
- added copper zone on F.Cu, net /Converter/SC_c1
- added copper zone on F.Cu, net /Converter/SC_c2
- added copper zone on F.Cu, net /Power /Vin
- added copper zone on B.Cu, net GND
- added copper zone on F.Cu, net GND
- added copper zone on F.Cu, net Net-(U1-SW)
Other:
- board text added: "Energy Flow Unit v1 Michał Borkowski 26.03.2024"

Commit message: Logs
Parts:
- C43, R35: moved to F.Cu
- moved R35 5.20 mm to (194.0, 82.2)
- turned C43 to 180 degrees
Routing:
- added copper zone on F.Cu, net Net-(U1-VIN)
- removed copper zone on B.Cu, net +12V
- removed copper zone on F.Cu, net /Power /Vin
Other:
- outline, holes or cut-outs redrawn

Commit message: Labels
Parts:
- moved J4 0.67 mm to (141.9, 136.2)
- moved C12 0.39 mm to (95.5, 67.5)
- moved R31 0.20 mm to (173.2, 117.2)
Connections:
- C14 pad 1: /MCU/XTAL_P -> /MCU/XTAL_N
- C15 pad 1: /MCU/XTAL_N -> /MCU/XTAL_P
Routing:
- net Net-(U1-SW): track 9.36 -> 16.8 mm
- net Net-(U1-VIN): track 56.0 -> 62.9 mm
- net +3.3V: track 387.8 -> 391.4 mm
