File: schematic-main.kicad_pcb (KiCad board)
At the start: 2 copper layers, 100 x 100 mm, 177 parts, among them IC1 LM76202QPWPRQ1, IC2 AD8544ARUZ-REEL, IC3 ACHS-7123-000E, IC4 ACHS-7121-000E, IC5 ACHS-7123-000E, IC6 LM5106MMX_NOPB, IC7 LM5106MMX_NOPB, IC8 MCP4018T-503E_LT, J1 Battery converter, J2 CAN, J3 FUEL CELL, J4 Joulemeter, J5 MOTOR CONTROLER, J6 SUPER CAPACITORS, P1 USB_C_Plug_USB2.0, Q1 CSD19531Q5AT, Q2 CSD19531Q5AT, Q3 CSD19531Q5AT, Q4 CSD19531Q5AT, U1 TPS62933, U2 USBLC6-2P6, U3 ESP32-S3FN8, U4 SN65HVD232, Y1 Crystal_GND24

Commit message: DRC Tested
Parts:
-  D6: renamed from D6
- C43, R35: moved to B.Cu
- CAN D4: renamed from D4
- MCU D5: renamed from D5
- moved C43 54.0 mm to (159.1, 113.2), turned to 0 degrees
- moved R35 37.7 mm to (165.4, 106.7), turned to -90 degrees
- renumbered R51 to (R51), TP4 to 12V, TP7 to 3.3V, TP6 to 5V, JP2 to BOOT, TP23 to D_P_W, TP24 to D_Pot_A, TP14 to FC_C, TP9 to I/O1, TP10 to I/O2, TP11 to I/O3, TP12 to I/O4, TP16 to MC_C, JP1 to RESET, TP15 to SC_C, JP3 to TEST, TP13 to TP_FC, TP19 to TP_SC
Routing:
- net /Converter/FC_c2: track 88.2 -> 101.5 mm, vias 2 -> 3
- net Net-(C43-Pad2): track 0.00 -> 6.29 mm
- net GND: track 1052.9 -> 1049.9 mm, vias 229 -> 218
- net /Converter/Bootstrap_B: track 139.3 -> 142.2 mm, vias 2 -> 3
- net /VBUS: track 113.9 -> 113.1 mm
Other:
- board text added: "+12V"
- board text added: "+3.3V"
- board text added: "+5V"
- board text added: "+J_SC"
- board text added: "A"
- board text added: "CAN"
- board text added: "CAN_HIGH"
- board text added: "CAN_LOW"
- board text added: "Digital_Potentiometer"
- board text added: "EN_A_test"
- board text added: "EN_B_test"
- board text added: "FC+"
- board text added: "FC_C_test"
- board text added: "FUEL_CELL"
- board text added: "GND"
- board text added: "I/O1"
- board text added: "I/O2"
- board text added: "I/O3"
- board text added: "I/O4"
- board text added: "JOULEMETER"
- board text added: "MC+"
- board text added: "MC_C_test"
- board text added: "MOTOR_CONTROLER"
- board text added: "POWER"
- board text added: "PWM_A_test"
- board text added: "PWM_B_test"
- board text added: "SC+"
- board text added: "SC_C_test"
- board text added: "SUPER_CAPACITORS"
- board text added: "VIN"
- board text added: "W"
- board text removed: "I/O 1 I/O 2"
- board text removed: "I/O 3 I/O 4"
